File: slave/slave-V11.brd (EAGLE design)
At the start: 28.9 x 40.6 mm, 23 parts, among them IC1 MPC9804, J1 TWIG-2.0-DIPD, U2 ATMEGA168

Commit message: a new master was born
Parts:
- removed C1: 0.1uF, SparkFun-Passives:0805
- removed C2: 1uF, SparkFun-Passives:0805
- removed R10, R3, R6, R7, R8, R9: 10K, SparkFun-Passives:0805
- removed SJ1, SJ2: SOLDERJUMPERNO, SparkFun-Passives:SJ_2S-NO
- added SW1: (no value), special:EDG-04
- IC1: value MPC9804 -> DS1820; device MCP9804:MSOP-8 -> DS1820:TO-92
- R2: value 10K -> 4.7K
- U1: value (none) -> INA169; device microbuilder:SOT23-8 -> SparkFun-AnalogIC:SOT23-5
- moved IC1 53.9 mm to (-38.1, 29.2)
- moved R1 50.6 mm to (-35.6, 19.1)
- moved R2 48.2 mm to (-26.7, 38.1)
- moved R5 47.9 mm to (-34.3, 38.1), turned to 0 degrees
- moved R4 42.0 mm to (-30.5, 38.1), turned to 0 degrees
- moved C4 39.6 mm to (-22.9, 38.1), turned to 0 degrees
- moved H1 39.5 mm to (-16.5, 31.8)
- moved U$1 35.9 mm to (-27.9, 19.1), turned to 0 degrees
- moved C3 35.1 mm to (-19.1, 38.1), turned to 0 degrees
- moved J1 34.7 mm to (-19.1, 3.81), turned to 0 degrees
- moved U1 34.2 mm to (-15.2, 38.1), turned to 0 degrees
- moved H2 29.3 mm to (-24.1, 31.8)
- moved U2 23.6 mm to (-17.8, 21.6)
Connections:
- removed net A0: IC1.P$7, R10.2, R2.2, SJ1.1, U1.7
- removed net A1: IC1.P$6, R3.2, R9.2, SJ2.1, U1.8
- removed net A2: IC1.P$5, R8.2
- removed net ALERT: IC1.P$3
- new net TEMP: IC1.2, R2.1
- net GND: now also IC1.1; no longer C1.2, C2.2, IC1.P$4, R10.1, R2.1, R3.1, R8.1, R9.1, U1.3
- net SCL: no longer IC1.P$2, R7.1, U1.5
- net SDA: no longer IC1.P$1, R6.1, U1.6
- net VCC: now also IC1.3, R2.2; no longer C1.1, C2.1, IC1.P$8, R6.2, R7.2, SJ1.2, SJ2.2, U1.4
- net VIN+: no longer U1.1
- net VIN-: no longer U1.2
Routing:
- net VCC: track 53.3 -> 0.00 mm
- net GND: track 33.8 -> 0.00 mm, vias 6 -> 0
- net A0: track 20.9 -> 0.00 mm
- net SCL: track 19.9 -> 0.00 mm
- net SDA: track 13.9 -> 0.00 mm, vias 2 -> 0
- net A1: track 10.5 -> 0.00 mm
- net VIN-: track 8.88 -> 0.00 mm
- net VIN+: track 8.35 -> 0.00 mm
- net A2: track 3.52 -> 0.00 mm
- net +12V: track 2.78 -> 0.00 mm
- removed copper zone on layer 1, net GND
- removed copper zone on layer 16, net N$1
- removed copper zone on layer 16, net N$2
- removed copper zone on layer 1, net VIN+
- removed copper zone on layer 1, net VIN-
Other:
- board size 28.9 x 40.6 mm -> 100 x 80 mm
