File: slave/slave-V11.sch (EAGLE design)
At the start: 24 parts, among them IC1 MPC9804, J1 TWIG-2.0-DIPD

Commit message: a new master was born
Parts:
- removed C1: 0.1uF, SparkFun-Passives:CAP0805
- removed C2: 1uF, SparkFun-Passives:CAP0805
- removed HOLE1, HOLE2: MOUNT-HOLE-0.138, holes:MOUNT-HOLE-0.138
- removed R10, R3, R6, R7, R8, R9: 10K, SparkFun-Passives:RESISTOR0805-RES
- removed SJ1, SJ2: SOLDERJUMPERNO, SparkFun-Passives:SOLDERJUMPERNO
- added SW1: (no value), special:SW_DIP-4
- added U2: ATMEGA168, SparkFun-DigitalIC:ATMEGA168
- IC1: value MPC9804 -> DS1820; device MCP9804:MPC9804 -> DS1820:DS1820
- R2: value 10K -> 4.7K
- U1: value (none) -> INA169; device microbuilder:INA219 -> SparkFun-AnalogIC:INA169
Connections:
- removed net A0: R10.2, R2.2, SJ1.1, U1.A0
- removed net A1: IC1.A1, R3.2, R9.2, SJ2.1, U1.A1
- removed net A2: IC1.A2, R8.2
- removed net ALERT: IC1.ALERT
- new net TEMP: IC1.DQ, R2.1
- net GND: now also IC1.GND; no longer C1.2, C2.2, R10.1, R2.1, R3.1, R8.1, R9.1, U1.GND
- net SCL: no longer IC1.SCL, R7.1, U1.SCL
- net SDA: no longer IC1.SDA, R6.1, U1.SDA
- net VCC: now also R2.2, U2.AREF, U2.AVCC, U2.VCC@1, U2.VCC@2; no longer C1.1, C2.1, R6.2, R7.2, SJ1.2, SJ2.2, U1.VCC
- net VIN+: no longer U1.VIN+
- net VIN-: no longer U1.VIN-
Other:
- moved on the sheet: C3, C4, H1, H2, R1, R2, U$1
