File: master/master-v11.brd (EAGLE design)
At the start: 58 x 59.7 mm, 48 parts

Commit message: Cambiado INA169 por ACS711 Cambiado conector de energia por molex 22-05
Parts:
- removed INA169: INA169, SparkFun-AnalogIC:SOT23-5
- removed JP2: M02JST-PTH-2, SparkFun-Connectors:JST-2-PTH
- removed SHUNT: 0.002, SparkFun-Resistors:1206
- added J1: 22-05-7028-02, con-molex:7395-02
- added U$3: ACS711, ACS711:SOIC8
- R13: value 82k -> 1k
- V_IN, V_OUT: value MOUNT-PAD-ROUND3.0 -> MOUNT-PAD-ROUND4.5; device holes:3,0-PAD -> holes:4,5-PAD
- moved C1 3.86 mm to (5.07, 10.9), turned to 0 degrees
- moved C4 3.75 mm to (1.90, 7.42), turned to 270 degrees
- moved C7 3.16 mm to (32.0, 45.9)
- moved R13 2.94 mm to (32.0, 47.9), turned to 0 degrees
- moved V_OUT 2.36 mm to (48.0, 54.0)
- moved V_IN 2.31 mm to (48.0, 39.0)
- moved C3 1.00 mm to (10.2, 17.5)
- moved C9 1.00 mm to (12.7, 17.5)
Connections:
- removed net VIN+: INA169.3, SHUNT.2, V_IN.B3,0
- removed net VIN-: INA169.4, SHUNT.1, V_OUT.B3,0
- new net N$69: R13.2, U$3.6
- new net N$71: U$3.1, U$3.2, V_IN.B4,5
- new net N$72: U$3.3, U$3.4, V_OUT.B4,5
- net 3.3V: now also C7.1, R13.1, U$3.8; no longer INA169.5
- net GND: now also J1.1, U$3.5; no longer INA169.2, JP2.1, R13.1
- net RAW: now also J1.2; no longer JP2.2
- net SENSOR_CURRENT: now also U$3.7; no longer C7.1, INA169.1, R13.2
Routing:
- net VIN-: track 12.5 -> 0.00 mm
- net VIN+: track 12.4 -> 0.00 mm
- net 3.3V: track 282.0 -> 287.5 mm
- net N$69: track 0.00 -> 5.23 mm
- net RAW: track 76.9 -> 79.6 mm
- net SENSOR_CURRENT: track 17.8 -> 20.3 mm

Commit message: render
PCB Black
Parts:
- added U$4: (no value), Logos:LOGO_ELIBATT2
Changed lines of the file:
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@@
 <?xml version="1.0" encoding="utf-8"?>
 <!DOCTYPE eagle SYSTEM "eagle.dtd">
-<eagle version="7.0.0">
+<eagle version="6.5.0">
 <drawing>
 <settings>
@@
 <setting verticaltext="up"/>
 </settings>
-<grid distance="0.5" unitdist="mm" unit="mm" style="lines" multiple="1" display="yes" altdistance="0.2" altunitdist="mm" altunit="mm"/>
+<grid distance="0.05" unitdist="inch" unit="mm" style="lines" multiple="1" display="yes" altdistance="0.005" altunitdist="inch" altunit="inch"/>
 <layers>
 <layer number="1" name="Top" color="4" fill="1" visible="yes" active="yes"/>
@@
 <layer number="23" name="tOrigins" color="15" fill="1" visible="yes" active="yes"/>
 <layer number="24" name="bOrigins" color="15" fill="1" visible="yes" active="yes"/>
-<layer number="25" name="tNames" color="7" fill="1" visible="no" active="yes"/>
+<layer number="25" name="tNames" color="7" fill="1" visible="yes" active="yes"/>
 <layer number="26" name="bNames" color="7" fill="1" visible="no" active="yes"/>
 <layer number="27" name="tValues" color="7" fill="1" visible="no" active="yes"/>
@@
 <layer number="36" name="bGlue" color="7" fill="5" visible="no" active="yes"/>
 <layer number="37" name="tTest" color="7" fill="1" visible="yes" active="yes"/>
-<layer number="38" name="bTest" color="7" fill="1" visible="no" active="yes"/>
+<layer number="38" name="bTest" color="7" fill="1" visible="yes" active="yes"/>
 <layer number="39" name="tKeepout" color="4" fill="11" visible="no" active="yes"/>
 <layer number="40" name="bKeepout" color="1" fill="11" visible="no" active="yes"/>
@@
 <layer number="220" name="220bmp" color="21" fill="1" visible="no" active="no"/>
 <layer number="221" name="221bmp" color="22" fill="1" visible="no" active="no"/>
-<layer number="222" name="222bmp" color="7" fill="1" visible="yes" active="yes"/>
 <layer number="223" name="223bmp" color="24" fill="1" visible="no" active="no"/>
 <layer number="224" name="224bmp" color="25" fill="1" visible="no" active="no"/>
@@
 <pass name="Default">
 <param name="RoutingGrid" value="50mil"/>
-<param name="AutoGrid" value="1"/>
-<param name="Efforts" value="0"/>
-<param name="TopRouterVariant" value="1"/>
 <param name="tpViaShape" value="round"/>
 <param name="PrefDir.1" value="|"/>
@@
 <elements>
 <element name="C2" library="rcl" package="C0805K" value="0.1uF" x="25.4" y="19.05" smashed="yes" rot="R270">
-<attribute name="NAME" x="26.675" y="19.85" size="1" layer="25" rot="R270"/>
+<attribute name="NAME" x="24.727" y="16.007" size="1" layer="25"/>
 <attribute name="VALUE" x="23.5" y="20.05" size="1.016" layer="27" rot="R270"/>
 </element>
@@
 <element name="TX" library="adafruit" package="CHIPLED_0805" value="RED" x="29.21" y="2.54" rot="R90"/>
 <element name="RX" library="adafruit" package="CHIPLED_0805" value="GREEN" x="33.02" y="2.54" rot="R90"/>
-<element name="R8" library="rcl" package="R0805" value="10k" x="29.21" y="19.05" rot="R270"/>
+<element name="R8" library="rcl" package="R0805" value="10k" x="29.21" y="19.05" smashed="yes" rot="R270">
+<attribute name="NAME" x="27.686" y="15.748" size="1.27" layer="25"/>
+<attribute name="VALUE" x="26.67" y="19.685" size="1.27" layer="27" rot="R270"/>
+</element>
 <element name="U$3" library="ACS711" package="SOIC8" value="ACS711" x="40.37" y="46.49" rot="R90"/>
 <element name="J1" library="con-molex" package="7395-02" value="22-05-7028-02" x="10.5" y="12.5">
@@
 <attribute name="OC_FARNELL" value="9731601" x="10.5" y="12.5" size="1.778" layer="27" display="off"/>
 </element>
+<element name="U$4" library="Logos" package="LOGO_ELIBATT2" value="" x="29.337" y="14.224"/>
 </elements>
 <signals>

Commit message: gerbes + BOM
add more tweaks
Parts:
- removed 3V3: AP1117E, v-reg:SOT223
- removed RTC: DS3231/SO, adafruit:SO16W
- removed U$3: ACS711, ACS711:SOIC8
- added ACS711: ACS711, ACS711:SOIC8
- added AP1117: AP1117E, v-reg:SOT223
- added DS3231: DS3231/SO, adafruit:SO16W
- moved OSC 2.08 mm to (26.7, 24.5)
- moved R8 1.80 mm to (27.9, 20.3)
- moved U$4 1.30 mm to (29.1, 15.5)
- moved ATMEGA1280 1.27 mm to (26.7, 35.6)
- moved BANCO 1.27 mm to (17.8, 52.1)
- moved BLE 1.27 mm to (29.2, 52.1)
- moved C 1.27 mm to (55.5, 40.6)
- moved C7 1.27 mm to (32.0, 47.2)
- moved GPS 1.27 mm to (6.35, 52.1)
- moved R11 1.27 mm to (39.4, 26.7)
- moved R13 1.27 mm to (32.0, 49.2)
- moved SD_L 1.27 mm to (41.3, 26.7)
- moved V_IN 1.27 mm to (48.0, 40.3)
- moved V_OUT 1.27 mm to (48.0, 55.3)
- moved TEMP 1.27 mm to (39.4, 16.5)
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Connections:
- net 3.3V: now also ACS711.8, AP1117.2, AP1117.4, DS3231.2; no longer 3V3.2, 3V3.4, RTC.2, U$3.8
- net GND: now also ACS711.5, AP1117.1, DS3231.10, DS3231.11, DS3231.12, DS3231.13, DS3231.5, DS3231.6, DS3231.7, DS3231.8, DS3231.9; no longer 3V3.1, RTC.10, RTC.11, RTC.12, RTC.13, RTC.5, RTC.6, RTC.7, RTC.8, RTC.9, U$3.5
- net MOSI: now also DS3231.15; no longer RTC.15
- net N$1: now also DS3231.14; no longer RTC.14
- net N$69: now also ACS711.6; no longer U$3.6
- net N$71: now also ACS711.1, ACS711.2; no longer U$3.1, U$3.2
- net N$72: now also ACS711.3, ACS711.4; no longer U$3.3, U$3.4
- net RAW: now also AP1117.3; no longer 3V3.3
- net SCK: now also DS3231.16; no longer RTC.16
- net SENSOR_CURRENT: now also ACS711.7; no longer U$3.7
Routing:
- net N$2: track 6.72 -> 5.52 mm
- net N$14: track 4.51 -> 3.56 mm
- net SENSOR_CURRENT: track 20.3 -> 21.1 mm
- net 3.3V: track 287.5 -> 286.8 mm
Other:
- board size 58 x 59.7 mm -> 58 x 61.2 mm
- board text added: "V1 1432"
- board text removed: "V1 1431"
