File: master/master-v11.sch (EAGLE design)
At the start: 46 parts

Commit message: Cambiado INA169 por ACS711 Cambiado conector de energia por molex 22-05
Parts:
- removed INA169: INA169, SparkFun-AnalogIC:INA169
- removed JP2: M02JST-PTH-2, SparkFun-Connectors:M02JST-PTH-2
- removed SHUNT: 0.002, SparkFun-Resistors:RESISTOR1206
- added J1: 22-05-7028-02, con-molex:22-05-7028-02
- added U$3: ACS711, ACS711:ACS711
- R13: value 82k -> 1k
- V_IN, V_OUT: value MOUNT-PAD-ROUND3.0 -> MOUNT-PAD-ROUND4.5; device holes:MOUNT-PAD-ROUND3.0 -> holes:MOUNT-PAD-ROUND4.5
Connections:
- removed net VIN+: INA169.VIN+, SHUNT.2, V_IN.MOUNT
- removed net VIN-: INA169.VIN-, SHUNT.1, V_OUT.MOUNT
- new net N$69: R13.2, U$3.FAULT
- new net N$71: U$3.IP+@1, U$3.IP+@2, V_IN.MOUNT
- new net N$72: U$3.IP-@3, U$3.IP-@4, V_OUT.MOUNT
- net 3.3V: now also C7.1, R13.1, U$3.VCC; no longer INA169.V+
- net GND: now also J1-1.S, U$3.GND; no longer INA169.GND, JP2.1, R13.1
- net RAW: now also J1-2.S; no longer JP2.2
- net SENSOR_CURRENT: now also U$3.VOUT; no longer C7.1, INA169.OUT, R13.2
Other:
- moved on the sheet: C7, R13, V_IN, V_OUT

Commit message: gerbes + BOM
add more tweaks
Parts:
- renumbered 3V3 to AP1117, RTC to DS3231, U$3 to ACS711
Changed lines of the file:
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@@
 <?xml version="1.0" encoding="utf-8"?>
 <!DOCTYPE eagle SYSTEM "eagle.dtd">
-<eagle version="7.0.0">
+<eagle version="6.5.0">
 <drawing>
 <settings>
@@
 <part name="GND6" library="SparkFun" deviceset="GND" device=""/>
 <part name="R3" library="rcl" deviceset="R-EU_" device="R0805" value="1K"/>
-<part name="RTC" library="adafruit" deviceset="DS3231" device="/SO"/>
+<part name="DS3231" library="adafruit" deviceset="DS3231" device="/SO"/>
 <part name="GND8" library="SparkFun" deviceset="GND" device=""/>
 <part name="ATMEGA1280" library="atmel-avr" deviceset="ATMEGA640/1280/2560" device="-A"/>
@@
 <part name="GND14" library="SparkFun" deviceset="GND" device=""/>
 <part name="FRAME1" library="SparkFun-Aesthetics" deviceset="FRAME-LEDGER" device=""/>
-<part name="3V3" library="v-reg" deviceset="AP1117" device="E"/>
+<part name="AP1117" library="v-reg" deviceset="AP1117" device="E"/>
 <part name="GND18" library="SparkFun" deviceset="GND" device=""/>
 <part name="R10" library="rcl" deviceset="R-EU_" device="R0805" value="10k"/>
@@
 <part name="RX" library="adafruit" deviceset="LED" device="CHIPLED_0805" value="GREEN"/>
 <part name="R8" library="rcl" deviceset="R-EU_" device="R0805" value="10k"/>
-<part name="U$3" library="ACS711" deviceset="ACS711" device=""/>
+<part name="ACS711" library="ACS711" deviceset="ACS711" device=""/>
 <part name="GND4" library="SparkFun" deviceset="GND" device=""/>
 <part name="SUPPLY11" library="SparkFun-Aesthetics" deviceset="3.3V" device=""/>
@@
 <instance part="GND6" gate="1" x="55.88" y="238.76"/>
 <instance part="R3" gate="G$1" x="160.02" y="109.22" rot="R90"/>
-<instance part="RTC" gate="G$1" x="25.4" y="60.96"/>
+<instance part="DS3231" gate="G$1" x="25.4" y="60.96"/>
 <instance part="GND8" gate="1" x="7.62" y="38.1"/>
 <instance part="ATMEGA1280" gate="G$1" x="205.74" y="167.64"/>
@@
 <instance part="FRAME1" gate="G$1" x="0" y="0"/>
 <instance part="FRAME1" gate="G$2" x="330.2" y="0"/>
-<instance part="3V3" gate="G$1" x="55.88" y="254"/>
+<instance part="AP1117" gate="G$1" x="55.88" y="254"/>
 <instance part="GND18" gate="1" x="162.56" y="215.9"/>
 <instance part="R10" gate="G$1" x="299.72" y="152.4"/>
@@
 <instance part="RX" gate="G$1" x="88.9" y="134.62" rot="R270"/>
 <instance part="R8" gate="G$1" x="154.94" y="248.92" rot="R90"/>
-<instance part="U$3" gate="G$1" x="309.88" y="254"/>
+<instance part="ACS711" gate="G$1" x="309.88" y="254"/>
 <instance part="GND4" gate="1" x="347.98" y="243.84"/>
 <instance part="SUPPLY11" gate="G$1" x="332.74" y="241.3" rot="R180"/>
@@
 <pinref part="GND6" gate="1" pin="GND"/>
 <wire x1="55.88" y1="241.3" x2="55.88" y2="246.38" width="0.1524" layer="91"/>
-<pinref part="3V3" gate="G$1" pin="GND"/>
-</segment>
-<segment>
-<pinref part="RTC" gate="G$1" pin="NC1"/>
+<pinref part="AP1117" gate="G$1" pin="GND"/>
+</segment>
+<segment>
+<pinref part="DS3231" gate="G$1" pin="NC1"/>
 <wire x1="10.16" y1="58.42" x2="7.62" y2="58.42" width="0.1524" layer="91"/>
 <wire x1="7.62" y1="58.42" x2="7.62" y2="55.88" width="0.1524" layer="91"/>
-<pinref part="RTC" gate="G$1" pin="NC3"/>
+<pinref part="DS3231" gate="G$1" pin="NC3"/>
 <wire x1="7.62" y1="55.88" x2="7.62" y2="53.34" width="0.1524" layer="91"/>
-<pinref part="RTC" gate="G$1" pin="NC2"/>
+<pinref part="DS3231" gate="G$1" pin="NC2"/>
 <wire x1="10.16" y1="55.88" x2="7.62" y2="55.88" width="0.1524" layer="91"/>
 <junction x="7.62" y="55.88"/>
-<pinref part="RTC" gate="G$1" pin="NC"/>
+<pinref part="DS3231" gate="G$1" pin="NC"/>
 <wire x1="10.16" y1="60.96" x2="7.62" y2="60.96" width="0.1524" layer="91"/>
 <wire x1="7.62" y1="60.96" x2="7.62" y2="58.42" width="0.1524" layer="91"/>
@@
 </segment>
 <segment>
-<pinref part="RTC" gate="G$1" pin="NC7"/>
+<pinref part="DS3231" gate="G$1" pin="NC7"/>
 <wire x1="40.64" y1="60.96" x2="43.18" y2="60.96" width="0.1524" layer="91"/>
 <wire x1="43.18" y1="60.96" x2="43.18" y2="58.42" width="0.1524" layer="91"/>
-<pinref part="RTC" gate="G$1" pin="NC6"/>
+<pinref part="DS3231" gate="G$1" pin="NC6"/>
 <wire x1="43.18" y1="58.42" x2="40.64" y2="58.42" width="0.1524" layer="91"/>
 <wire x1="43.18" y1="58.42" x2="43.18" y2="55.88" width="0.1524" layer="91"/>
 <junction x="43.18" y="58.42"/>
-<pinref part="RTC" gate="G$1" pin="NC5"/>
+<pinref part="DS3231" gate="G$1" pin="NC5"/>
 <wire x1="43.18" y1="55.88" x2="40.64" y2="55.88" width="0.1524" layer="91"/>
 <wire x1="43.18" y1="55.88" x2="43.18" y2="53.34" width="0.1524" layer="91"/>
 <junction x="43.18" y="55.88"/>
-<pinref part="RTC" gate="G$1" pin="NC4"/>
+<pinref part="DS3231" gate="G$1" pin="NC4"/>
 <wire x1="43.18" y1="53.34" x2="40.64" y2="53.34" width="0.1524" layer="91"/>
-<pinref part="RTC" gate="G$1" pin="GND"/>
+<pinref part="DS3231" gate="G$1" pin="GND"/>
 <wire x1="40.64" y1="63.5" x2="43.18" y2="63.5" width="0.1524" layer="91"/>
 <wire x1="43.18" y1="63.5" x2="43.18" y2="60.96" width="0.1524" layer="91"/>
@@
 <segment>
 <pinref part="GND1" gate="1" pin="GND"/>
-<pinref part="U$3" gate="G$1" pin="GND"/>
+<pinref part="ACS711" gate="G$1" pin="GND"/>
 <wire x1="325.12" y1="246.38" x2="325.12" y2="251.46" width="0.1524" layer="91"/>
 <wire x1="325.12" y1="251.46" x2="322.58" y2="251.46" width="0.1524" layer="91"/>
@@
 </segment>
 <segment>
-<pinref part="RTC" gate="G$1" pin="SCL"/>
+<pinref part="DS3231" gate="G$1" pin="SCL"/>
 <wire x1="40.64" y1="71.12" x2="45.72" y2="71.12" width="0.1524" layer="91"/>
 <label x="43.18" y="71.12" size="1.778" layer="95"/>
@@
 </segment>
 <segment>
-<pinref part="RTC" gate="G$1" pin="SDA"/>
+<pinref part="DS3231" gate="G$1" pin="SDA"/>
 <wire x1="40.64" y1="68.58" x2="45.72" y2="68.58" width="0.1524" layer="91"/>
 <label x="43.18" y="68.58" size="1.778" layer="95"/>
@@
 <wire x1="45.72" y1="248.92" x2="45.72" y2="254" width="0.1524" layer="91"/>
 <junction x="45.72" y="254"/>
-<pinref part="3V3" gate="G$1" pin="IN"/>
+<pinref part="AP1117" gate="G$1" pin="IN"/>
 <pinref part="J1" gate="-2" pin="S"/>
 </segment>
@@
 <net name="N$1" class="0">
 <segment>
-<pinref part="RTC" gate="G$1" pin="VBAT"/>
+<pinref part="DS3231" gate="G$1" pin="VBAT"/>
 <pinref part="BAT" gate="G$1" pin="+"/>
 <wire x1="40.64" y1="66.04" x2="50.8" y2="66.04" width="0.1524" layer="91"/>
@@
 <junction x="71.12" y="254"/>
 <pinref part="SUPPLY1" gate="G$1" pin="3.3V"/>
-<pinref part="3V3" gate="G$1" pin="OUT"/>
+<pinref part="AP1117" gate="G$1" pin="OUT"/>
 </segment>
 <segment>
@@
 </segment>
 <segment>
-<pinref part="RTC" gate="G$1" pin="VCC"/>
+<pinref part="DS3231" gate="G$1" pin="VCC"/>
 <wire x1="10.16" y1="68.58" x2="7.62" y2="68.58" width="0.1524" layer="91"/>
 <wire x1="7.62" y1="68.58" x2="7.62" y2="78.74" width="0.1524" layer="91"/>
@@
 </segment>
 <segment>
-<pinref part="U$3" gate="G$1" pin="VCC"/>
+<pinref part="ACS711" gate="G$1" pin="VCC"/>
 <pinref part="SUPPLY5" gate="G$1" pin="3.3V"/>
 <wire x1="347.98" y1="259.08" x2="322.58" y2="259.08" width="0.1524" layer="91"/>
@@
 <segment>
 <label x="340.36" y="256.54" size="1.27" layer="95" rot="R270" xref="yes"/>
-<pinref part="U$3" gate="G$1" pin="VOUT"/>
+<pinref part="ACS711" gate="G$1" pin="VOUT"/>
 <wire x1="322.58" y1="256.54" x2="340.36" y2="256.54" width="0.1524" layer="91"/>
 </segment>
@@
 <net name="N$69" class="0">
 <segment>
-<pinref part="U$3" gate="G$1" pin="FAULT"/>
+<pinref part="ACS711" gate="G$1" pin="FAULT"/>
 <wire x1="322.58" y1="254" x2="332.74" y2="254" width="0.1524" layer="91"/>
 <pinref part="R13" gate="G$1" pin="2"/>
@@
 <net name="N$71" class="0">
 <segment>
-<pinref part="U$3" gate="G$1" pin="IP+@2"/>
+<pinref part="ACS711" gate="G$1" pin="IP+@2"/>
 <wire x1="287.02" y1="269.24" x2="287.02" y2="259.08" width="0.1524" layer="91"/>
 <wire x1="287.02" y1="259.08" x2="287.02" y2="256.54" width="0.1524" layer="91"/>
 <wire x1="287.02" y1="256.54" x2="294.64" y2="256.54" width="0.1524" layer="91"/>
-<pinref part="U$3" gate="G$1" pin="IP+@1"/>
+<pinref part="ACS711" gate="G$1" pin="IP+@1"/>
 <wire x1="294.64" y1="259.08" x2="287.02" y2="259.08" width="0.1524" layer="91"/>
 <pinref part="V_IN" gate="G$1" pin="MOUNT"/>
@@
 <net name="N$72" class="0">
 <segment>
-<pinref part="U$3" gate="G$1" pin="IP-@3"/>
+<pinref part="ACS711" gate="G$1" pin="IP-@3"/>
 <wire x1="287.02" y1="241.3" x2="287.02" y2="251.46" width="0.1524" layer="91"/>
 <wire x1="287.02" y1="251.46" x2="287.02" y2="254" width="0.1524" layer="91"/>
 <wire x1="287.02" y1="254" x2="294.64" y2="254" width="0.1524" layer="91"/>
-<pinref part="U$3" gate="G$1" pin="IP-@4"/>
+<pinref part="ACS711" gate="G$1" pin="IP-@4"/>
 <wire x1="294.64" y1="251.46" x2="287.02" y2="251.46" width="0.1524" layer="91"/>
 <pinref part="V_OUT" gate="G$1" pin="MOUNT"/>
