File: Hardware/master/master-v12_36V.brd (EAGLE design)
At the start: 58 x 61.2 mm, 48 parts, among them J1 22-05-7028-02, X1 USB-MB-H

Commit message: BOM Master V12 + gerbers
Parts:
- R14: value 10k -> 39.7k
Connections:
- removed net CD: MICROSD.CD1
- removed net VCC: AP1117.2, AP1117.4, C1.1, C3.1, C9.A, FT232RL.20, X1.VBUS
- new net VCC1: C3.1, C9.A, FT232RL.20, X1.VBUS
- new net VCCIO: FT232RL.4
- net 3.3V: now also AP1117.2, AP1117.4, C1.1; no longer FT232RL.4
Routing:
- net VCC: track 50.8 -> 0.00 mm, vias 3 -> 0
- net VCC1: track 0.00 -> 16.8 mm, vias 0 -> 1
- net GND: track 24.5 -> 12.0 mm, vias 16 -> 14
- net 3.3V: track 257.8 -> 249.2 mm, vias 9 -> 4
- net AUX_CURRENT: track 3.21 -> 11.2 mm
- net SCK: track 74.2 -> 76.1 mm
- net COMM_TX: track 37.4 -> 36.4 mm
- net SCL: track 49.3 -> 50.2 mm
- net MISO: track 69.2 -> 68.6 mm
