File: Hardware/master/master-v12_36V.sch (EAGLE design)
At the start: 45 parts, among them J1 22-05-7028-02, X1 USB-MB-H

Commit message: BOM Master V12 + gerbers
Parts:
- ACS711: MPN ACS711KLCTR-25AB-T -> (none); OC_NEWARK 24T5972 -> (none)
- AP1117: MPN AP1117E33G-13 -> (none); OC_NEWARK 79R5845 -> (none)
- ATMEGA1280, BANCO, BLE, DS3231, FRAME1, FT232RL, GPS, ISP, MICROSD, S1, V_IN, V_OUT, X1: OC_NEWARK unknown -> (none)
- BAT: MF SANYO, HAWKER, PANASONIC BATTE -> (none); MPN CR1220 -> (none); OC_NEWARK 15C6530 -> (none)
- C1, C4, C9: MPN 0805ZD106KAT2A -> (none); OC_NEWARK 96M1311 -> (none)
- C11, C2, C3, C6, C7: MPN MC0603B104K500CT -> (none); OC_NEWARK 06R4927 -> (none)
- DBG_L, SD_L: MPN 150080BS75000 -> (none); OC_NEWARK 95W3799 -> (none)
- OSC: MPN PBRC8.00HR50X000 -> (none); OC_NEWARK 23M7097 -> (none)
- PWR, TX: MPN KPT-2012SRC-J4 -> (none); OC_NEWARK 88W4951 -> (none)
- R1, R11, R2, R3, R5, R6, R7: MF VISHAY/DALE -> (none); MPN CRCW08051K00FKTA -> (none); OC_NEWARK 05F1507 -> (none)
- R10, R13, R16, R8: MF VISHAY/DALE -> (none); MPN CRCW080510K0FKTA -> (none); OC_NEWARK 05F1511 -> (none)
- R14: value 10k -> 39.7k; MF VISHAY/DALE -> (none); MPN CRCW080510K0FKTA -> (none); OC_NEWARK 05F1511 -> (none)
- R15: MF VISHAY/DALE -> (none); MPN CRCW08053K30FKTA -> (none); OC_NEWARK 48F4423 -> (none)
- RX: MPN 150080VS75000 -> (none); OC_NEWARK 95W3803 -> (none)
- TEMP: MPN MCP9808-E/MS -> (none); OC_NEWARK 89T8871 -> (none)
Connections:
- removed net CD: MICROSD.SHIELD@2
- removed net VCC: AP1117.OUT, C1.1, C3.1, C9.+, FT232RL.VCC, X1.VBUS
- new net VCC1: C3.1, C9.+, FT232RL.VCC, X1.VBUS
- net 3.3V: now also AP1117.OUT, C1.1; no longer FT232RL.VCCIO
